Commit message: x500 position controller training

File: resources/robots/x500/x500.urdf (robot description, URDF)
Before this commit: robot quadrotor, 9 links, 8 joints
Links:
- link arm_motor_0: geometry visual cylinder length=0.24607315985291853 radius=0.01
- link arm_motor_1: geometry visual cylinder length=0.24607315985291853 radius=0.01
- link arm_motor_2: geometry visual cylinder length=0.24607315985291853 radius=0.01
- link arm_motor_3: geometry visual cylinder length=0.24607315985291853 radius=0.01
- link base_link: geometry collision sphere radius=0.29607315985291854; visual sphere radius=0.05
- link motor_0: geometry visual cylinder length=0.05 radius=0.01
- link motor_1: geometry visual cylinder length=0.05 radius=0.01
- link motor_2: geometry visual cylinder length=0.05 radius=0.01
- link motor_3: geometry visual cylinder length=0.05 radius=0.01
Joints:
- joint base_link_to_arm_motor_0: origin xyz=0.087 -0.087 0.0 rpy=-1.5707963267948968 2.220446049250313e-16 -2.3561944901923453 -> xyz=0.087 -0.087 0.0 rpy=-1.5707963267948966 2.220446049250313e-16 -2.356194490192345
- joint base_link_to_arm_motor_1: origin xyz=-0.087 -0.087 0.0 rpy=1.5707963267948968 2.220446049250313e-16 -0.7853981633974482 -> xyz=-0.087 -0.087 0.0 rpy=1.5707963267948966 2.220446049250313e-16 -0.7853981633974483
- joint base_link_to_arm_motor_2: origin xyz=-0.087 0.087 0.0 rpy=1.5707963267948968 0.0 -2.3561944901923453 -> xyz=-0.087 0.087 0.0 rpy=1.5707963267948966 0.0 -2.356194490192345
- joint base_link_to_arm_motor_3: origin xyz=0.087 0.087 0.0 rpy=-1.5707963267948968 0.0 -0.7853981633974482 -> xyz=0.087 0.087 0.0 rpy=-1.5707963267948966 0.0 -0.7853981633974483
- joint base_link_to_motor_0: origin xyz=0.174 -0.174 0.06 rpy=0.0 0.0 0.0 -> xyz=0.174 -0.174 0.0 rpy=0.0 0.0 0.0
- joint base_link_to_motor_1: origin xyz=-0.174 -0.174 0.06 rpy=0.0 0.0 0.0 -> xyz=-0.174 -0.174 0.0 rpy=0.0 0.0 0.0
- joint base_link_to_motor_2: origin xyz=-0.174 0.174 0.06 rpy=0.0 0.0 0.0 -> xyz=-0.174 0.174 0.0 rpy=0.0 0.0 0.0
- joint base_link_to_motor_3: origin xyz=0.174 0.174 0.06 rpy=0.0 0.0 0.0 -> xyz=0.174 0.174 0.0 rpy=0.0 0.0 0.0
